File: newer/longBoard.kicad_pcb (KiCad board)
At the start: 2 copper layers, 82.6 x 166.4 mm, 67 parts, among them Q1 IRLZ34N, Q2 IRLZ34N, Q3 IRLZ34N, Q4 IRLZ34N, Q5 IRLZ34N, Q6 IRLZ34N, Q7 IRLZ34N, Q8 IRLZ34N, U1 Teensy3.5, U10 HCPL3120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

Commit message: first version of the long board concept, its not great but it looks ok from a quick look
Parts:
- moved Serial1 91.5 mm to (207.0, 105.4), turned to 180 degrees
- moved CAN1 81.9 mm to (207.0, 115.6), turned to 180 degrees
- moved Serial3 70.1 mm to (207.0, 127.0), turned to 180 degrees
- moved PPM9 14.9 mm to (221.0, 204.5), turned to 90 degrees
- moved PPM10 2.54 mm to (221.0, 207.0)
Routing:
- net Net-(CAN1-Pad1): track 7.62 -> 203.9 mm, vias 0 -> 2
- net Net-(R21-Pad1): track 6.01 -> 134.0 mm
- net +24V: track 408.8 -> 529.5 mm
- net /Sheet58E8F73D/cleanGND: track 332.6 -> 441.0 mm, vias 1 -> 2
- net Net-(Serial1-Pad3): track 106.5 -> 3.81 mm
- net GND: track 186.7 -> 287.0 mm
- net Net-(CAN1-Pad3): track 102.4 -> 4.86 mm
- net Net-(R25-Pad1): track 6.01 -> 103.5 mm
- net Net-(Serial1-Pad2): track 99.6 -> 3.81 mm
- net Net-(R23-Pad1): track 51.6 -> 144.4 mm
- net Net-(CAN1-Pad2): track 94.1 -> 4.86 mm
- net Net-(R18-Pad1): track 24.2 -> 112.5 mm
- net Net-(R19-Pad1): track 25.8 -> 113.9 mm
- net Net-(PPM10-Pad1): track 0.00 -> 86.1 mm
- net Net-(PPM9-Pad1): track 0.00 -> 85.9 mm
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
Commit message: more updates
Parts:
- added R29: R, robotlibary:logoA1, F.Cu at (247.0, 269.1)
Routing:
- net Net-(CAN1-Pad1): track 203.9 -> 205.2 mm, vias 2 -> 0
- net /Sheet58E8F73D/cleanGND: track 441.0 -> 440.5 mm
