File: newer/secondGo.kicad_pcb (KiCad board)
At the start: 2 copper layers, 50 parts, among them Q1 IRLZ34N, Q2 IRLZ34N, Q3 IRLZ34N, Q4 IRLZ34N, Q5 IRLZ34N, Q6 IRLZ34N, Q7 IRLZ34N, Q8 IRLZ34N, U1 TEENSY3.1, U10 HCPL3120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

Commit message: move the two versions in to to directorys
Parts:
- U11: value TRACO_TEL_DCDC -> TRACO_DCDC_TEL_3-2411; footprint Housings_DIP:DIP-24_W15.24mm -> robotlibary:traco_TEL_3-2411
- U3: value TRACO_TEL_DCDC -> TRACO_DCDC_TVN_5-4815WI; footprint Housings_DIP:DIP-24_W15.24mm -> robotlibary:traco_TVN_5-4815WI
Connections:
- U1 pad 10: Net-(U1-Pad10) -> (no net)
- U1 pad 11: Net-(U1-Pad11) -> (no net)
- U1 pad 12: Net-(U1-Pad12) -> (no net)
- U1 pad 13: Net-(U1-Pad13) -> (no net)
- U1 pad 14: Net-(U1-Pad14) -> (no net)
- U1 pad 15: Net-(U1-Pad15) -> (no net)
- U1 pad 16: Net-(U1-Pad16) -> (no net)
- U1 pad 17: Net-(U1-Pad17) -> (no net)
- U1 pad 18: Net-(U1-Pad18) -> (no net)
- U1 pad 19: Net-(U1-Pad19) -> (no net)
- U1 pad 2: Net-(U1-Pad2) -> (no net)
- U1 pad 20: Net-(U1-Pad20) -> (no net)
- U1 pad 3: Net-(U1-Pad3) -> (no net)
- U1 pad 31: Net-(U1-Pad31) -> (no net)
- U1 pad 32: Net-(U1-Pad32) -> (no net)
- U1 pad 34: Net-(U1-Pad34) -> (no net)
- U1 pad 35: Net-(U1-Pad35) -> (no net)
- U1 pad 36: Net-(U1-Pad36) -> (no net)
- U1 pad 37: Net-(U1-Pad37) -> (no net)
- U1 pad 38: Net-(U1-Pad38) -> (no net)
- U1 pad 39: Net-(U1-Pad39) -> (no net)
- U1 pad 4: Net-(U1-Pad4) -> (no net)
- U1 pad 40: Net-(U1-Pad40) -> (no net)
- U1 pad 41: Net-(U1-Pad41) -> (no net)
- U1 pad 42: Net-(U1-Pad42) -> (no net)
- U1 pad 43: Net-(U1-Pad43) -> (no net)
- U1 pad 44: Net-(U1-Pad44) -> (no net)
- U1 pad 45: Net-(U1-Pad45) -> (no net)
- U1 pad 46: Net-(U1-Pad46) -> (no net)
- U1 pad 47: Net-(U1-Pad47) -> (no net)
- U1 pad 48: Net-(U1-Pad48) -> (no net)
- U1 pad 49: Net-(U1-Pad49) -> (no net)
- U1 pad 50: Net-(U1-Pad50) -> (no net)
- U1 pad 51: Net-(U1-Pad51) -> (no net)
- U1 pad 9: Net-(U1-Pad9) -> (no net)
- U10 pad 1: Net-(U10-Pad1) -> (no net)
- U10 pad 4: Net-(U10-Pad4) -> (no net)
- U10 pad 6: Net-(U10-Pad6) -> (no net)
- U11 pad 1: +24V -> Net-(U1-Pad33)
- U11 pad 10: Net-(U1-Pad33) -> +24V
- U11 pad 11: /Sheet58E8F73D/cleanGND -> GND
- U11 pad 12: GND -> /Sheet58E8F73D/cleanGND
- U2 pad 1: Net-(U2-Pad1) -> (no net)
- U2 pad 4: Net-(U2-Pad4) -> (no net)
- U2 pad 6: Net-(U2-Pad6) -> (no net)
- U3 pad 1: +24V -> Net-(Pressure1-Pad1)
- U3 pad 10: Net-(Pressure1-Pad1) -> (no net)
- U3 pad 11: /Sheet58E8F73D/cleanGND -> (no net)
- U3 pad 12: GND -> (no net)
- U3 pad 14: (no net) -> GND
- U3 pad 15: (no net) -> +24V
- U4 pad 1: Net-(U4-Pad1) -> (no net)
- U4 pad 4: Net-(U4-Pad4) -> (no net)
- U4 pad 6: Net-(U4-Pad6) -> (no net)
- U5 pad 1: Net-(U5-Pad1) -> (no net)
- U5 pad 4: Net-(U5-Pad4) -> (no net)
- U5 pad 6: Net-(U5-Pad6) -> (no net)
- U6 pad 1: Net-(U6-Pad1) -> (no net)
- U6 pad 4: Net-(U6-Pad4) -> (no net)
- U6 pad 6: Net-(U6-Pad6) -> (no net)
- U7 pad 1: Net-(U7-Pad1) -> (no net)
- U7 pad 4: Net-(U7-Pad4) -> (no net)
- U7 pad 6: Net-(U7-Pad6) -> (no net)
- U8 pad 1: Net-(U8-Pad1) -> (no net)
- U8 pad 4: Net-(U8-Pad4) -> (no net)
- U8 pad 6: Net-(U8-Pad6) -> (no net)
- U9 pad 1: Net-(U9-Pad1) -> (no net)
- U9 pad 4: Net-(U9-Pad4) -> (no net)
- U9 pad 6: Net-(U9-Pad6) -> (no net)

Commit message: trying to see if ican get it to fin in alexs space
Parts:
- added R17: R, Resistors_THT:R_Axial_DIN0207_L6.3mm_D2.5mm_P10.16mm_Horizontal, F.Cu at (75.1, 163.1)
- added R18: R, Resistors_THT:R_Axial_DIN0207_L6.3mm_D2.5mm_P10.16mm_Horizontal, F.Cu at (61.2, 163.1)
- added R19: R, Resistors_THT:R_Axial_DIN0207_L6.3mm_D2.5mm_P10.16mm_Horizontal, F.Cu at (47.2, 163.1)
- added R20: R, Resistors_THT:R_Axial_DIN0207_L6.3mm_D2.5mm_P10.16mm_Horizontal, F.Cu at (75.1, 168.2)
- added R21: R, Resistors_THT:R_Axial_DIN0207_L6.3mm_D2.5mm_P10.16mm_Horizontal, F.Cu at (33.2, 163.1)
- added R22: R, Resistors_THT:R_Axial_DIN0207_L6.3mm_D2.5mm_P10.16mm_Horizontal, F.Cu at (61.2, 168.2)
- added R23: R, Resistors_THT:R_Axial_DIN0207_L6.3mm_D2.5mm_P10.16mm_Horizontal, F.Cu at (19.3, 163.1)
- added R24: R, Resistors_THT:R_Axial_DIN0207_L6.3mm_D2.5mm_P10.16mm_Horizontal, F.Cu at (47.2, 168.2)
- added R25: R, Resistors_THT:R_Axial_DIN0207_L6.3mm_D2.5mm_P10.16mm_Horizontal, F.Cu at (5.28, 163.1)
- added R26: R, Resistors_THT:R_Axial_DIN0207_L6.3mm_D2.5mm_P10.16mm_Horizontal, F.Cu at (33.2, 168.2)
- added R27: R, Resistors_THT:R_Axial_DIN0207_L6.3mm_D2.5mm_P10.16mm_Horizontal, F.Cu at (19.3, 168.2)
- added R28: R, Resistors_THT:R_Axial_DIN0207_L6.3mm_D2.5mm_P10.16mm_Horizontal, F.Cu at (5.28, 168.2)
- R10, R11, R12, R13, R14, R15, R16, R9: footprint Diodes_THT:D_5W_P5.08mm_Vertical_AnodeUp -> robotlibary:Selinoid
- moved R9 209.9 mm to (269.5, 168.7), turned to 0 degrees
- moved D1 201.2 mm to (274.6, 176.3), turned to 180 degrees
- moved Retract1 196.0 mm to (2.66, 156.6)
- moved R1 190.4 mm to (264.4, 204.2), turned to 0 degrees
- moved R10 189.5 mm to (255.5, 168.7), turned to 0 degrees
- moved Q1 185.1 mm to (267.0, 199.1), turned to 0 degrees
- moved U2 182.6 mm to (265.7, 218.2), turned to 90 degrees
- moved R13 179.6 mm to (269.4, 163.1), turned to 180 degrees
- moved Targeting1 178.2 mm to (15.4, 156.6)
- moved D2 177.5 mm to (260.6, 176.3), turned to 180 degrees
- moved D3 173.5 mm to (246.6, 176.3), turned to 180 degrees
- moved R11 169.4 mm to (241.6, 168.7), turned to 0 degrees
- moved R2 168.9 mm to (250.5, 204.2), turned to 0 degrees
- moved Q2 166.3 mm to (253.0, 199.1), turned to 0 degrees
- moved D5 166.0 mm to (264.4, 156.7), turned to 0 degrees
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Connections:
- Retract1 pad 2: Net-(Retract1-Pad2) -> Net-(R25-Pad2)
- Spare1 pad 2: Net-(Spare1-Pad2) -> Net-(R21-Pad2)
- Targeting1 pad 2: Net-(Targeting1-Pad2) -> Net-(R23-Pad2)
- U1 pad 21: Net-(Pressure1-Pad2) -> Net-(R17-Pad1)
- U1 pad 22: Net-(Presure2-Pad2) -> Net-(R18-Pad1)
- U1 pad 23: Net-(Presure3-Pad2) -> Net-(R19-Pad1)
- U1 pad 24: Net-(Spare1-Pad2) -> Net-(R21-Pad1)
- U1 pad 25: Net-(Targeting1-Pad2) -> Net-(R23-Pad1)
- U1 pad 26: Net-(Retract1-Pad2) -> Net-(R25-Pad1)
Routing:
- net +24V: track 0.00 -> 504.0 mm
- net GND: track 0.00 -> 321.5 mm
- net /Sheet58E8F73D/cleanGND: track 0.00 -> 157.5 mm
- net Net-(Pressure1-Pad1): track 0.00 -> 86.9 mm
- net Net-(D6-Pad2): track 0.00 -> 38.3 mm
- net Net-(D1-Pad2): track 0.00 -> 38.3 mm
- net Net-(D8-Pad2): track 0.00 -> 38.3 mm
- net Net-(D7-Pad2): track 0.00 -> 38.3 mm
- net Net-(D5-Pad2): track 0.00 -> 38.3 mm
- net Net-(D2-Pad2): track 0.00 -> 38.3 mm
- net Net-(D4-Pad2): track 0.00 -> 38.3 mm
- net Net-(D3-Pad2): track 0.00 -> 38.3 mm
- net Net-(Presure2-Pad2): track 0.00 -> 13.8 mm
- net Net-(Presure3-Pad2): track 0.00 -> 13.7 mm
- net Net-(Pressure1-Pad2): track 0.00 -> 12.5 mm
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
Commit message: first version with the 3.5
Parts:
- removed U11: TRACO_DCDC_TEL_3-2411, robotlibary:traco_TEL_3-2411
- removed U3: TRACO_DCDC_TVN_5-4815WI, robotlibary:traco_TVN_5-4815WI
- added CAN1: CONN_01X04, Pin_Headers:Pin_Header_Straight_1x04_Pitch2.54mm, F.Cu at (210.8, 139.7)
- added PPM10: CONN_01X03, Pin_Headers:Pin_Header_Angled_1x03_Pitch2.54mm, F.Cu at (226.1, 147.3)
- added PPM9: CONN_01X03, Pin_Headers:Pin_Header_Angled_1x03_Pitch2.54mm, F.Cu at (224.8, 99.1)
- added Reg24v1: TRACO_DCDC_TVN_5-4815WI, robotlibary:traco_TVN_5-4815WI, F.Cu at (228.6, 175.3)
- added Reg5v1: TRACO_DCDC_TEL_3-2411, robotlibary:traco_TEL_3-2411, F.Cu at (203.2, 167.6)
- added Serial1: CONN_01X04, Pin_Headers:Pin_Header_Straight_1x04_Pitch2.54mm, F.Cu at (203.2, 139.7)
- added Serial3: CONN_01X04, Pin_Headers:Pin_Header_Straight_1x04_Pitch2.54mm, F.Cu at (207.0, 139.7)
- BT1: footprint BoardEdgebattery:WSBattery -> robotlibary:WSBattery
- Pressure1, Presure2, Presure3, Retract1, Spare1, Targeting1: footprint wsPot:Potentiometer_Trimmer_WS_Vertical_Px5.0mm_Py10.0mm -> Pin_Headers:Pin_Header_Angled_1x03_Pitch2.54mm
- R10, R11, R12, R13, R14, R15, R16, R9: footprint robotlibary:Selinoid -> robotlibary:Value
- U1: value TEENSY3.1 -> Teensy3.5; footprint Teensy:Teensy30_31_32_LC -> Teensy:Teensy35_36
- moved R28 184.0 mm to (189.2, 162.6), turned to 270 degrees
- moved R23 181.4 mm to (195.6, 205.7), turned to 90 degrees
- moved R25 181.4 mm to (186.7, 162.6), turned to 270 degrees
- moved Retract1 179.4 mm to (181.6, 168.9)
- moved R27 177.8 mm to (193.0, 205.7), turned to 90 degrees
- moved Targeting1 173.7 mm to (181.6, 207.0)
- moved R26 158.4 mm to (189.2, 195.6), turned to 270 degrees
- moved Spare1 156.9 mm to (181.6, 199.4)
- moved R21 156.9 mm to (186.7, 195.6), turned to 270 degrees
- moved R24 147.7 mm to (194.3, 181.6), turned to 270 degrees
- moved R19 145.8 mm to (191.8, 181.6), turned to 270 degrees
- moved Presure3 141.4 mm to (181.6, 191.8)
- moved R22 128.8 mm to (189.2, 181.6), turned to 270 degrees
- moved R18 126.9 mm to (186.7, 181.6), turned to 270 degrees
- moved Presure2 126.1 mm to (181.6, 184.2)
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Connections:
- U1 pad 10: (no net) -> Net-(Serial3-Pad2)
- U1 pad 11: (no net) -> Net-(PPM9-Pad1)
- U1 pad 12: (no net) -> Net-(PPM10-Pad1)
- U1 pad 2: (no net) -> Net-(Serial1-Pad3)
- U1 pad 21: Net-(R17-Pad1) -> (no net)
- U1 pad 22: Net-(R18-Pad1) -> (no net)
- U1 pad 23: Net-(R19-Pad1) -> (no net)
- U1 pad 24: Net-(R21-Pad1) -> (no net)
- U1 pad 25: Net-(R23-Pad1) -> (no net)
- U1 pad 26: Net-(R25-Pad1) -> (no net)
- U1 pad 27: /Sheet58E8F73D/chanel8 -> (no net)
- U1 pad 28: /Sheet58E8F73D/chanel7 -> (no net)
- U1 pad 29: /Sheet58E8F73D/chanel6 -> (no net)
- U1 pad 3: (no net) -> Net-(Serial1-Pad2)
- U1 pad 30: /Sheet58E8F73D/changel5 -> (no net)
- U1 pad 33: Net-(U1-Pad33) -> /Sheet58E8F73D/chanel1
- U1 pad 34: (no net) -> /Sheet58E8F73D/chanel8
- U1 pad 35: (no net) -> /Sheet58E8F73D/chanel2
- U1 pad 41: (no net) -> Net-(R17-Pad1)
- U1 pad 42: (no net) -> Net-(R18-Pad1)
- U1 pad 43: (no net) -> Net-(R19-Pad1)
- U1 pad 44: (no net) -> Net-(R21-Pad1)
- U1 pad 45: (no net) -> Net-(R23-Pad1)
- U1 pad 46: (no net) -> Net-(R25-Pad1)
- U1 pad 48: (no net) -> /Sheet58E8F73D/chanel7
- U1 pad 49: (no net) -> /Sheet58E8F73D/chanel6
- U1 pad 5: /Sheet58E8F73D/chanel1 -> Net-(CAN1-Pad3)
- U1 pad 50: (no net) -> /Sheet58E8F73D/changel5
- U1 pad 6: /Sheet58E8F73D/chanel2 -> Net-(CAN1-Pad2)
- U1 pad 9: (no net) -> Net-(Serial3-Pad3)
Routing:
- net /Sheet58E8F73D/cleanGND: track 157.5 -> 518.9 mm, vias 0 -> 1
- net Net-(CAN1-Pad1): track 0.00 -> 124.1 mm
- net Net-(R23-Pad1): track 5.08 -> 98.3 mm
- net /Sheet58E8F73D/chanel2: track 0.00 -> 85.8 mm
- net /Sheet58E8F73D/chanel4: track 0.00 -> 80.9 mm
- net Net-(PPM9-Pad1): track 0.00 -> 78.4 mm
- net Net-(R21-Pad1): track 5.08 -> 80.9 mm
- net /Sheet58E8F73D/chanel1: track 0.00 -> 75.3 mm
- net Net-(CAN1-Pad3): track 0.00 -> 71.4 mm, vias 0 -> 2
- net /Sheet58E8F73D/chanel3: track 0.00 -> 71.0 mm
- net Net-(CAN1-Pad2): track 0.00 -> 66.4 mm, vias 0 -> 2
- net Net-(Serial1-Pad3): track 0.00 -> 65.6 mm, vias 0 -> 2
- net Net-(PPM10-Pad1): track 0.00 -> 61.3 mm
- net Net-(Serial1-Pad2): track 0.00 -> 61.3 mm, vias 0 -> 2
- net /Sheet58E8F73D/chanel8: track 0.00 -> 58.8 mm
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Other:
- board outline added: 115.6 x 118.1 mm
- net class powerTracks added: clearance 0.254, trace_width 0.254, via_dia 0.889, via_drill 0.635

Commit message: little fixes
Routing:
- net +24V: track 463.7 -> 542.2 mm
Other:
- board size 115.6 x 118.1 mm -> 115.6 x 119.4 mm

Commit message: more little fixes
Routing:
- net /Sheet58E8F73D/cleanGND: track 518.9 -> 541.0 mm
Changed lines of the file:
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@@
     (thickness 1.6)
     (drawings 8)
-    (tracks 433)
+    (tracks 437)
     (zones 0)
     (modules 67)
@@
   (segment (start 232.41 158.75) (end 232.41 179.07) (width 0.254) (layer B.Cu) (net 34))
   (segment (start 232.41 179.07) (end 236.22 182.88) (width 0.254) (layer B.Cu) (net 34))
+  (segment (start 189.23 205.74) (end 190.5 205.74) (width 0.254) (layer F.Cu) (net 35))
+  (segment (start 190.5 205.74) (end 191.77 207.01) (width 0.254) (layer F.Cu) (net 35))
+  (segment (start 191.77 207.01) (end 198.12 207.01) (width 0.254) (layer F.Cu) (net 35))
+  (segment (start 198.12 207.01) (end 198.12 191.77) (width 0.254) (layer F.Cu) (net 35))
+  (segment (start 203.2 147.32) (end 198.12 147.32) (width 0.254) (layer F.Cu) (net 35))
+  (segment (start 198.12 147.32) (end 196.85 147.32) (width 0.254) (layer F.Cu) (net 35))
+  (segment (start 198.12 182.88) (end 198.12 147.32) (width 0.254) (layer F.Cu) (net 35))
   (segment (start 200.66 208.28) (end 203.2 208.28) (width 1) (layer B.Cu) (net 35))
   (segment (start 203.2 208.28) (end 203.2 190.5) (width 1) (layer B.Cu) (net 35))
@@
   (via (at 189.23 208.28) (size 0.889) (drill 0.635) (layers F.Cu B.Cu) (net 35))
   (segment (start 179.07 201.93) (end 179.07 208.28) (width 1) (layer F.Cu) (net 35))
-  (segment (start 189.23 205.74) (end 189.23 208.28) (width 0.254) (layer F.Cu) (net 35))
   (segment (start 228.6 167.64) (end 228.6 152.4) (width 0.254) (layer F.Cu) (net 35))
   (segment (start 228.6 149.86) (end 228.6 152.4) (width 0.254) (layer F.Cu) (net 35))
@@
   (segment (start 191.77 172.72) (end 189.23 172.72) (width 0.254) (layer B.Cu) (net 35))
   (segment (start 198.12 191.77) (end 198.12 182.88) (width 0.254) (layer F.Cu) (net 35))
-  (segment (start 198.12 182.88) (end 198.12 147.32) (width 0.254) (layer F.Cu) (net 35))
   (segment (start 194.787882 182.88) (end 198.12 182.88) (width 0.254) (layer F.Cu) (net 35))
   (segment (start 191.292118 182.88) (end 194.787882 182.88) (width 0.254) (layer F.Cu) (net 35))
@@
   (segment (start 179.07 201.93) (end 179.07 194.31) (width 1) (layer F.Cu) (net 35))
   (segment (start 181.61 201.93) (end 179.07 201.93) (width 0.254) (layer F.Cu) (net 35))
-  (segment (start 203.2 147.32) (end 196.85 147.32) (width 0.254) (layer F.Cu) (net 35))
   (segment (start 196.85 147.32) (end 196.85 97.79) (width 0.254) (layer F.Cu) (net 35))
   (segment (start 196.85 97.79) (end 179.07 97.79) (width 0.254) (layer F.Cu) (net 35))

Commit message: more updates
Changed lines of the file:
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@@
   (general
     (links 157)
-    (no_connects 6)
-    (area 0 0 0 0)
+    (no_connects 5)
+    (area 170.930999 92.659999 288.340001 214.489)
     (thickness 1.6)
     (drawings 8)
-    (tracks 437)
+    (tracks 440)
     (zones 0)
     (modules 67)
@@
   (segment (start 246.38 123.19) (end 246.38 124.46) (width 0.254) (layer F.Cu) (net 7))
   (segment (start 246.38 124.46) (end 243.84 127) (width 0.254) (layer F.Cu) (net 7))
+  (segment (start 260.35 133.35) (end 260.35 119.38) (width 3) (layer B.Cu) (net 8))
+  (segment (start 260.35 119.38) (end 260.35 105.41) (width 3) (layer B.Cu) (net 8))
+  (segment (start 275.59 119.38) (end 260.35 119.38) (width 1) (layer B.Cu) (net 8))
+  (segment (start 260.35 175.26) (end 260.35 161.29) (width 3) (layer B.Cu) (net 8))
+  (segment (start 260.35 161.29) (end 260.35 147.32) (width 3) (layer B.Cu) (net 8))
+  (segment (start 275.834344 161.559448) (end 260.619448 161.559448) (width 1) (layer B.Cu) (net 8))
+  (segment (start 260.619448 161.559448) (end 260.35 161.29) (width 0.254) (layer B.Cu) (net 8))
   (segment (start 245.11 194.31) (end 245.11 205.74) (width 0.254) (layer B.Cu) (net 8))
   (segment (start 275.59 203.2) (end 260.35 203.2) (width 1) (layer B.Cu) (net 8))
@@
   (segment (start 260.35 189.23) (end 260.35 175.26) (width 3) (layer B.Cu) (net 8))
   (segment (start 275.59 189.23) (end 260.35 189.23) (width 1) (layer B.Cu) (net 8))
-  (segment (start 260.35 175.26) (end 260.35 147.32) (width 3) (layer B.Cu) (net 8))
   (segment (start 275.59 175.26) (end 260.35 175.26) (width 1) (layer B.Cu) (net 8))
-  (segment (start 275.834344 161.559448) (end 260.619448 161.559448) (width 1) (layer B.Cu) (net 8))
   (segment (start 260.35 147.32) (end 260.35 133.35) (width 3) (layer B.Cu) (net 8))
   (segment (start 275.59 147.32) (end 260.35 147.32) (width 1) (layer B.Cu) (net 8))
-  (segment (start 260.35 133.35) (end 260.35 105.41) (width 3) (layer B.Cu) (net 8))
   (segment (start 275.59 133.35) (end 260.35 133.35) (width 1) (layer B.Cu) (net 8))
-  (segment (start 275.59 119.38) (end 260.35 119.38) (width 1) (layer B.Cu) (net 8))
   (segment (start 260.35 105.41) (end 275.59 105.41) (width 1) (layer B.Cu) (net 8))
   (segment (start 250.220078 205.74) (end 260.35 205.74) (width 3) (layer B.Cu) (net 8))
